File: hardware-q2-placement/2_POWER.kicad_sch (KiCad schematic)
At the start: 38 parts, among them U14 STC3115AIQT, U3 DSCB_BQ25895RTW, U4 TLV62568DBVR, U5 ME6211C18M5G-N, U6 GEK100

Commit message: feat: relocate harness connectors and refine Q2 enclosure
Parts:
- H2: value (none) -> BM03B-ACHSS-GAN-ETF; footprint MP3_Source:HDR-TH_3P-P2.54-V-M -> MP3_Source:JST_ACH_BM03B-ACHSS-GAN-ETF_1x03-1MP_P1.20mm_Vertical; Supplier Part C2937625 -> (none)
Changed lines of the file:
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@@
 			)
 		)
-		(property "Value" ""
+		(property "Value" "BM03B-ACHSS-GAN-ETF"
 			(at 76.2 86.36 0)
 			(show_name no)
@@
 				)
 			)
+			(hide yes)
 		)
-		(property "Footprint" "MP3_Source:HDR-TH_3P-P2.54-V-M"
+		(property "Footprint" "MP3_Source:JST_ACH_BM03B-ACHSS-GAN-ETF_1x03-1MP_P1.20mm_Vertical"
 			(at 76.2 86.36 0)
 			(hide yes)
@@
 			)
 		)
-		(property "Datasheet" ""
+		(property "Datasheet" "https://www.jst-mfg.com/product/pdf/eng/eACH.pdf"
 			(at 76.2 86.36 0)
 			(hide yes)
@@
 			)
 		)
-		(property "Description" ""
+		(property "Description" "Battery; pin 1 VBAT, pin 2 BAT_TS, pin 3 GBAT"
 			(at 76.2 86.36 0)
 			(hide yes)
@@
 			)
 		)
-		(property "Supplier Part" "C2937625"
+		(property "Supplier Part" ""
 			(at 76.2 86.36 0)
 			(hide yes)

Commit message: fix: restore schematic links and refine PCB component placement
Parts:
- removed R10: 0R/NC, MP3_Source:R0402, symbol MP3_Source:电阻
Connections:
- net BAT_TS: now also R13.2, R14.2, R15.2, R16.2, U3.11 (TS)
