File: hardware-q2-placement/5_MOTOR.kicad_sch (KiCad schematic)
At the start: 6 parts, among them U11 DRV2605LDGSR

Commit message: feat: relocate harness connectors and refine Q2 enclosure
Parts:
- H1: value (none) -> BM02B-ACHSS-GAN-ETF; footprint MP3_Source:HDR-TH_2P-P2.54-V-F -> MP3_Source:JST_ACH_BM02B-ACHSS-GAN-ETF_1x02-1MP_P1.20mm_Vertical; Supplier Part C49661 -> (none)
Changed lines of the file:
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@@
 			)
 		)
-		(property "Value" ""
+		(property "Value" "BM02B-ACHSS-GAN-ETF"
 			(at 189.23 63.5 0)
 			(show_name no)
@@
 				)
 			)
+			(hide yes)
 		)
-		(property "Footprint" "MP3_Source:HDR-TH_2P-P2.54-V-F"
+		(property "Footprint" "MP3_Source:JST_ACH_BM02B-ACHSS-GAN-ETF_1x02-1MP_P1.20mm_Vertical"
 			(at 189.23 63.5 0)
 			(hide yes)
@@
 			)
 		)
-		(property "Datasheet" ""
+		(property "Datasheet" "https://www.jst-mfg.com/product/pdf/eng/eACH.pdf"
 			(at 189.23 63.5 0)
 			(hide yes)
@@
 			)
 		)
-		(property "Description" ""
+		(property "Description" "LRA motor; pin 1 OUT_N, pin 2 OUT_P"
 			(at 189.23 63.5 0)
 			(hide yes)
@@
 			)
 		)
-		(property "Supplier Part" "C49661"
+		(property "Supplier Part" ""
 			(at 189.23 63.5 0)
 			(hide yes)
