File: hardware-q2-placement/hardware.kicad_pcb (KiCad board)
At the start: 6 copper layers, 46 x 76 mm, 126 parts, among them CN1 PJ-342B-TX-SMT, U1 RX8130CE:BB, U11 DRV2605LDGSR, U12 CH343P, U14 STC3115AIQT, U15 LSM6DS3TR-C, U16 PAM2804AAB010, U17 SGM7229YMS10G/TR, U2 CS43131-CNZ, U3 DSCB_BQ25895RTW, U4 TLV62568DBVR, U5 ME6211C18M5G-N, U6 GEK100, U7 PCA9306DQER, U8 SN74LV4T125RGYR, U9 ESP32-S31-WROOM-3-N16R16V, X1 26MHz

Commit message: feat: relocate harness connectors and refine Q2 enclosure
Parts:
- H1: value ~ -> BM02B-ACHSS-GAN-ETF; footprint MP3_Source:HDR-TH_2P-P2.54-V-F -> MP3_Source:JST_ACH_BM02B-ACHSS-GAN-ETF_1x02-1MP_P1.20mm_Vertical
- H2: value ~ -> BM03B-ACHSS-GAN-ETF; footprint MP3_Source:HDR-TH_3P-P2.54-V-M -> MP3_Source:JST_ACH_BM03B-ACHSS-GAN-ETF_1x03-1MP_P1.20mm_Vertical
- moved H1 11.6 mm to (130.0, 113.0), turned to -90 degrees
- moved H2 7.05 mm to (142.0, 109.0), turned to -90 degrees

Commit message: fix: restore schematic links and refine PCB component placement
Parts:
- removed R10: 0R/NC, MP3_Source:R0402
- C28: moved to B.Cu
- C53, C54, C6, C7, R42, R7, R8, U1: moved to F.Cu
- moved R21 10.8 mm to (139.2, 97.2), turned to 180 degrees
- moved U6 10.3 mm to (116.5, 91.0)
- moved C44 10.0 mm to (127.5, 96.0), turned to -90 degrees
- moved C3 9.92 mm to (115.8, 88.0), turned to 180 degrees
- moved R1 9.89 mm to (144.0, 106.5), turned to 90 degrees
- moved C36 7.85 mm to (138.2, 104.0), turned to 0 degrees
- moved L3 7.57 mm to (124.5, 111.0), turned to 0 degrees
- moved R44 7.08 mm to (125.8, 117.5), turned to -90 degrees
- moved C4 6.90 mm to (120.2, 117.2)
- moved C58 6.88 mm to (121.5, 111.2)
- moved C55 6.60 mm to (131.0, 75.8), turned to 90 degrees
- moved R8 6.18 mm to (141.8, 88.8)
- moved R42 5.50 mm to (141.8, 91.2), turned to 90 degrees
- moved R22 5.39 mm to (136.0, 104.0), turned to 180 degrees
- moved C53 5.20 mm to (140.0, 92.5)
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Connections:
- R13 pad 2: Net-(U3-TS) -> BAT_TS
- R14 pad 2: Net-(U3-TS) -> BAT_TS
- U3 pad 11: Net-(U3-TS) -> BAT_TS
