File: hardware-q2/10_TOUCH_WHEEL.kicad_sch (KiCad schematic)
At the start: 7 parts, among them CN3 HX-XH2.54-2PWZ-B, U11 DRV2605LDGSR

Commit message: feat: save finalized module mainboard and fabrication review
Parts:
- removed ?: (no value), ProPrj_esp-easyedapro:, symbol ProPrj_esp-easyedapro:Drawing-Symbol_A4
- removed C4, C5: 1uF, ProPrj_esp-easyedapro:, symbol ProPrj_esp-easyedapro:cl05b104ko5nnnc_2
- removed C58: 100nF, ProPrj_esp-easyedapro:, symbol ProPrj_esp-easyedapro:cl05b104ko5nnnc_2
- removed CN3: HX-XH2.54-2PWZ-B, ProPrj_esp-easyedapro:CONN-TH_2P-P2.50_HX-XH2.54-2PWZ-B, symbol ProPrj_esp-easyedapro:HX-XH2.54-2PWZ-B
- removed L3: BLM18KG601SN1D, ProPrj_esp-easyedapro:L0603, symbol ProPrj_esp-easyedapro:BLM18KG601SN1D
- removed U11: DRV2605LDGSR, ProPrj_esp-easyedapro:VSSOP-10_L3.0-W3.0-P0.50-LS4.9-BL, symbol ProPrj_esp-easyedapro:DRV2605LDGSR
- added ?: (no value), ProPrj_esp-easyedapro:, symbol ProPrj_esp-easyedapro:Drawing-Symbol_A4
- added C59: 100nF, ProPrj_esp-easyedapro:C0402, symbol ProPrj_esp-easyedapro:Capacitance
- added FPC1: HC-FPC-05-10-12RLTAG, ProPrj_esp-easyedapro:FPC-SMD_12P-P0.50_HCTL_HC-FPC-05-10-12RLTAG, symbol ProPrj_esp-easyedapro:HC-FPC-05-10-12RLTAG
Connections:
- net GND: now also C59.2, FPC1.1, FPC1.12, FPC1.13, FPC1.14
- new net TOUCH_I2C_SCL: FPC1.4
- new net TOUCH_I2C_SDA: FPC1.3
- new net TOUCH_INT#: FPC1.5
- new net TOUCH_POWER#: FPC1.11
- new net TOUCH_RESET#: FPC1.6
- new net VCC_TW: C59.1, FPC1.2
- no-connect marks 0 -> 4
