File: hardware-q2/1_MCU.kicad_sch (KiCad schematic)
At the start: 24 parts, among them Q1 S8050 (optional, not fitted), Q2 S8050 (optional, not fitted), U9 ESP32-S31-WROOM-3-N16R16V

Commit message: feat: save finalized module mainboard and fabrication review
Parts:
- removed C39, C41: 1uF, MP3_Source:C0402, symbol MP3_Source:Capacitance
- removed C40: 100nF, MP3_Source:C0402, symbol MP3_Source:Capacitance
- removed Q1, Q2: S8050 (optional, not fitted), symbol MP3_Source:NPN
- removed R20, R25, R26, R29, R30, R35, R36, R37, R38, R39, R43, R44, R7, R8: 10K, MP3_Source:R0402, symbol MP3_Source:电阻
- removed R23, R24: 10K, symbol MP3_Source:电阻
- removed R27, R28: 0/NC, MP3_Source:R0402, symbol MP3_Source:电阻
- removed U9: ESP32-S31-WROOM-3-N16R16V, MP3_Source:CONN-SMD_ESP32-S31-WROOM-3, symbol MP3_Source:ESP32-S31-WROOM-3-N16R16V_C55371223
- added ?: (no value), ProPrj_esp-easyedapro:, symbol ProPrj_esp-easyedapro:Drawing-Symbol_A4
- added C13, C40: 100nF, ProPrj_esp-easyedapro:C0402, symbol ProPrj_esp-easyedapro:Capacitance
- added C39, C41: 1uF, ProPrj_esp-easyedapro:C0402, symbol ProPrj_esp-easyedapro:Capacitance
- added Q1, Q2: (no value), ProPrj_esp-easyedapro:S8050_SOT-23, symbol ProPrj_esp-easyedapro:NPN
- added R10, R20, R22, R23, R24, R25, R26, R29, R30, R35, R36, R37, R38, R39, R42, R43, R44, R45, R46, R6, R7, R8: 10K, ProPrj_esp-easyedapro:R1206, symbol ProPrj_esp-easyedapro:电阻
- added R27, R28: 0/NC, ProPrj_esp-easyedapro:R1206, symbol ProPrj_esp-easyedapro:电阻
- added U10: W25Q16JVSSIQ, ProPrj_esp-easyedapro:SOIC-8_L5.3-W5.3-P1.27-LS8.0-BL, symbol ProPrj_esp-easyedapro:W25Q16JVSSIQTR
- added U9: ESP32-S31-WROOM-3-N16R16V, ProPrj_esp-easyedapro:CONN-SMD_ESP32-S31-WROOM-3, symbol ProPrj_esp-easyedapro:ESP32-S31-WROOM-3-N16R16V_C55371223
Connections:
- net CH343P_UART_DTR: now also Q2.2, R23.1, R28.2
- net CH343P_UART_RTS: now also Q1.2, R24.1, R27.1
- net ESP32S31_EN: now also C39.1, Q1.3, R27.2, R29.1, U9.5 (EN)
- net ESP_BOOT1: now also R20.2, R28.1, U9.71 (IO61)
- net ESP_BOOT2: now also R25.2, U9.70 (IO60)
- net ESP_FLASH_CLK: now also U10.6 (CLK), U9.17 (IO11)
- net ESP_FLASH_CS: now also U10.1 (/CS), U9.20 (IO14)
- net ESP_FLASH_DI: now also U10.5 (DI/IO0), U9.18 (IO12)
- net ESP_FLASH_DO: now also U10.2 (DO/IO1), U9.15 (IO9)
- net ESP_FLASH_HOLD: now also U10.7 (IO3), U9.16 (IO10)
- net ESP_FLASH_WP: now also U10.3 (IO2), U9.19 (IO13)
- net ESP_I2C2_SCL: now also R45.2, U9.66 (IO56)
- net ESP_I2C2_SDA: now also R46.2, U9.65 (IO55)
- net ESP_IO1: now also U9.9 (IO1)
- net ESP_IO19: now also U9.25 (IO19)
- net ESP_IO33: now also R10.2, R22.2, U9.42 (IO33)
- net ESP_IO34: now also R42.1, U9.43 (IO34)
- net ESP_IO35: now also R6.2, U9.44 (IO35)
- net ESP_IO4: now also U9.10 (IO4)
- net ESP_IO40: now also R44.2, U9.51 (IO40)
- net ESP_IO45: now also U9.55 (IO45)
- net ESP_IO46: now also U9.56 (IO46)
- net ESP_IO47: now also U9.57 (IO47)
- net ESP_IO5: now also U9.11 (IO5)
- net ESP_IO54: now also U9.64 (IO54)
- net ESP_IO57: now also U9.67 (IO57)
- net ESP_SPI2_CLK: now also U9.58 (IO48)
- net ESP_SPI2_CS: now also U9.59 (IO49)
- net ESP_SPI2_D0: now also U9.63 (IO53)
- net ESP_SPI2_D1: now also U9.61 (IO51)
- net ESP_SPI2_D2: now also U9.62 (IO52)
- net ESP_SPI2_D3: now also U9.60 (IO50)
- net ESP_TF_CLK: now also U9.31 (SD_CLK)
- net ESP_TF_CMD: now also R39.2, U9.32 (SD_CMD)
- net ESP_TF_DAT0: now also R38.2, U9.27 (SD_D0)
- net ESP_TF_DAT1: now also R35.2, U9.28 (SD_D1)
- net ESP_TF_DAT2: now also R36.2, U9.29 (SD_D2)
- net ESP_TF_DAT3: now also R37.2, U9.30 (SD_D3)
- net ESP_USB_DN: now also U9.41 (USB_DM)
- net ESP_USB_DP: now also U9.40 (USB_DP)
- net GND: now also C13.2, C39.2, C40.2, C41.2, R22.1, R44.1, U10.4 (GND), U9.1 (GND), U9.2 (GND), U9.26 (GND), U9.47 (GND), U9.48 (GND), U9.72 (GND), U9.73 (GND), U9.74 (GND), U9.75 (GND), U9.76 (GND), U9.77 (GND), U9.78 (GND), U9.79 (GND), U9.80 (GND), U9.81 (GND), U9.82 (GND), U9.83 (GND), U9.84 (GND), U9.85 (GND), U9.86 (GND), U9.87 (GND), U9.88 (GND), U9.89 (GND), U9.90 (GND), U9.92 (GND), U9.93 (GND), U9.94 (GND), U9.95 (GND), U9.96 (GND), U9.97 (GND), U9.98 (GND), U9.99 (GND)
- net VCC_3V3: now also C13.1, C40.1, C41.1, R10.1, R20.1, R25.1, R26.1, R29.2, R30.1, R35.1, R36.1, R37.1, R38.1, R39.1, R42.2, R43.1, R45.1, R46.1, R6.1, R7.1, R8.1, U10.8 (VCC), U9.3 (3V3), U9.4 (3V3)
- new net: Q1.1, R23.2
- new net: Q2.1, R24.2
- new net ESP32S31_BOOT: Q2.3
- new net ESP_I2C_SCL: R7.2, U9.45 (IO36)
- new net ESP_I2C_SDA: R8.2, U9.46 (IO37)
- new net ESP_I2S_LRCK: U9.21 (IO15)
- new net ESP_I2S_SCLK: U9.24 (IO18)
- new net ESP_I2S_SDIN: U9.22 (IO16)
- new net ESP_IO17: U9.23 (IO17)
- new net ESP_IO38: R43.2, U9.49 (IO38)
- new net ESP_IO39: U9.50 (IO39)
- new net ESP_IO42: U9.52 (IO42)
- new net ESP_IO43: U9.53 (IO43)
- new net ESP_IO44: U9.54 (IO44)
- new net ESP_LP_I2C_SCL: R26.2, U9.12 (IO6)
- new net ESP_LP_I2C_SDA: R30.2, U9.13 (IO7)
- new net ESP_UART_RX0: U9.69 (RX0)
- new net ESP_UART_TX0: U9.68 (TX0)
- no-connect marks 14 -> 7
Other:
- note added: "USB CH340 UART"
- note added: "USB DEBUG"
- note added: "USB OTG"
- company: ESP32-S31 MP3 -> (none)
- title: ESP32-S31 controller -> (none)
