File: hardware-q2/2_POWER.kicad_sch (KiCad schematic)
At the start: 38 parts, among them U14 STC3115AIQT, U3 DSCB_BQ25895RTW, U4 TLV62568DBVR, U5 ME6211C18M5G-N, U6 GEK100

Commit message: feat: save finalized module mainboard and fabrication review
Parts:
- removed C1: 10uF, MP3_Source:C0603_1_C1, symbol MP3_Source:Capacitance
- removed C10: 10uF, MP3_Source:C0603_1_C10, symbol MP3_Source:Capacitance
- removed C11: 47nF, MP3_Source:C0402, symbol MP3_Source:Capacitance
- removed C12: 10uF, MP3_Source:C0603_1_C12, symbol MP3_Source:Capacitance
- removed C13: 10uF, symbol MP3_Source:Capacitance
- removed C14: 1uF, MP3_Source:C0603_1_C14, symbol MP3_Source:Capacitance
- removed C15: 10uF, MP3_Source:C0603_1_C15, symbol MP3_Source:Capacitance
- removed C16: 47uF, MP3_Source:C0805, symbol MP3_Source:Capacitance
- removed C2: 10uF, MP3_Source:C0603_1_C2, symbol MP3_Source:Capacitance
- removed C3: 100nF, MP3_Source:C0402, symbol MP3_Source:Capacitance
- removed C30, C31: 1uF, MP3_Source:C0402_1, symbol MP3_Source:capacitance_2
- removed C43: 220nF, MP3_Source:C0402, symbol MP3_Source:Capacitance
- removed C9: 4.7uF, MP3_Source:C0603_1_C9, symbol MP3_Source:Capacitance
- removed D2: B5817W, MP3_Source:SOD-123_L2.8-W1.8-LS3.7-RD, symbol MP3_Source:B5817W_C181205
- removed H2: (no value), MP3_Source:HDR-TH_3P-P2.54-V-M, symbol MP3_Source:HDR-M_2.54_1x3P
- removed L1, L2: 2.2uH, MP3_Source:IND-SMD_L2.0-W1.6, symbol MP3_Source:WPN201610M2R2MT
- removed R1: 10mΩ, MP3_Source:R1206, symbol MP3_Source:RE1206F1R010
- removed R10, R34: 0R/NC, MP3_Source:R0402, symbol MP3_Source:电阻
- removed R11, R12, R4, R5: 100K, MP3_Source:R0402, symbol MP3_Source:电阻
- removed R13: 5K23, MP3_Source:R0402, symbol MP3_Source:电阻
- removed R14: 30K1, MP3_Source:R0402, symbol MP3_Source:电阻
- removed R15, R16: 10K, symbol MP3_Source:电阻
- removed R2, R33: 1K, MP3_Source:R0402, symbol MP3_Source:电阻
- removed R3: 22K1, MP3_Source:R0402, symbol MP3_Source:电阻
- removed R9: 700R, MP3_Source:R0402, symbol MP3_Source:电阻
- removed U14: STC3115AIQT, MP3_Source:DFN-10_L3.0-W2.0-P0.50-BL, symbol MP3_Source:STC3115AIQT
- removed U3: DSCB_BQ25895RTW, MP3_Source:WQFN-24_L4.0-W4.0-P0.50-TL-EP2.7, symbol MP3_Source:DSCB_BQ25895RTW
- removed U4: TLV62568DBVR, MP3_Source:SOT-23-5_L3.0-W1.7-P0.95-LS2.8-BR, symbol MP3_Source:TLV62568DBVR
- removed U5: ME6211C18M5G-N, MP3_Source:SOT-23-5_L3.0-W1.7-P0.95-LS2.8-BR_1, symbol MP3_Source:ME6211C18M5G-N
- removed U6: GEK100, MP3_Source:SOT-23-6_L2.9-W1.6-P0.95-LS2.8-BL-2, symbol MP3_Source:GEK100
- added ?: (no value), ProPrj_esp-easyedapro:, symbol ProPrj_esp-easyedapro:Drawing-Symbol_A4
- added C1, C10, C12, C15, C2, C62: 10uF, ProPrj_esp-easyedapro:C0402, symbol ProPrj_esp-easyedapro:Capacitance
- added C11: 47nF, ProPrj_esp-easyedapro:C0402, symbol ProPrj_esp-easyedapro:Capacitance
- added C14: 1uF, ProPrj_esp-easyedapro:C0402, symbol ProPrj_esp-easyedapro:Capacitance
- added C16: 47uF, ProPrj_esp-easyedapro:C0402, symbol ProPrj_esp-easyedapro:Capacitance
- added C3: 100nF, ProPrj_esp-easyedapro:C0402, symbol ProPrj_esp-easyedapro:Capacitance
- added C30, C31: 1uF, ProPrj_esp-easyedapro:, symbol ProPrj_esp-easyedapro:capacitance_2
- added C43, C61: 220nF, ProPrj_esp-easyedapro:C0402, symbol ProPrj_esp-easyedapro:Capacitance
- added C9: 4.7uF, ProPrj_esp-easyedapro:C0402, symbol ProPrj_esp-easyedapro:Capacitance
- added CN2: HX-XH2.54-3PWZ-B, ProPrj_esp-easyedapro:CONN-TH_3P-P2.50_BX-HA2.54-3PWZ, symbol ProPrj_esp-easyedapro:HX-XH2.54-3PWZ-B
- added D2: B5817W, ProPrj_esp-easyedapro:SOD-123_L2.8-W1.8-LS3.7-RD, symbol ProPrj_esp-easyedapro:B5817W_C181205
- added L1, L2: 2.2uH, ProPrj_esp-easyedapro:IND-SMD_L2.0-W1.6, symbol ProPrj_esp-easyedapro:WPN201610M2R2MT
- added R1: 10mΩ, ProPrj_esp-easyedapro:R1206, symbol ProPrj_esp-easyedapro:RE1206F1R010
- added R11, R12, R4, R5: 100K, ProPrj_esp-easyedapro:R1206, symbol ProPrj_esp-easyedapro:电阻
- added R13: 5K23, ProPrj_esp-easyedapro:R1206, symbol ProPrj_esp-easyedapro:电阻
- added R14: 30K1, ProPrj_esp-easyedapro:R1206, symbol ProPrj_esp-easyedapro:电阻
- added R15, R16: 10K, ProPrj_esp-easyedapro:R1206, symbol ProPrj_esp-easyedapro:电阻
- added R2, R33: 1K, ProPrj_esp-easyedapro:R1206, symbol ProPrj_esp-easyedapro:电阻
- added R3: 22K1, ProPrj_esp-easyedapro:R1206, symbol ProPrj_esp-easyedapro:电阻
- added R34: 0R, ProPrj_esp-easyedapro:R1206, symbol ProPrj_esp-easyedapro:电阻
- added R9: 700R, ProPrj_esp-easyedapro:R1206, symbol ProPrj_esp-easyedapro:电阻
- added U14: STC3115AIQT, ProPrj_esp-easyedapro:DFN-10_L3.0-W2.0-P0.50-BL, symbol ProPrj_esp-easyedapro:STC3115AIQT
- added U3: DSCB_BQ25895RTW, ProPrj_esp-easyedapro:DSCB:WQFN-24-1EP_4x4mm_P0.5mm_EP2.6x2.6mm, symbol ProPrj_esp-easyedapro:DSCB_BQ25895RTW
- added U4: TLV62568DBVR, ProPrj_esp-easyedapro:SOT-23-5_L3.0-W1.7-P0.95-LS2.8-BR, symbol ProPrj_esp-easyedapro:TLV62568DBVR
- added U5: ME6211C18M5G-N, ProPrj_esp-easyedapro:SOT-23-5_L3.0-W1.7-P0.95-LS2.8-BR_1, symbol ProPrj_esp-easyedapro:ME6211C18M5G-N
- added U6: GEK100, ProPrj_esp-easyedapro:SOT-23-6_L2.9-W1.6-P0.95-LS2.8-BL-2, symbol ProPrj_esp-easyedapro:GEK100
Connections:
- net BAT_TS: now also CN2.2, R13.2, R14.2, R15.2, R16.2
- net BQ25895_CHG_EN#: now also R11.2
- net BQ25895_OTG_EN: now also R12.2
- net GBAT: now also CN2.3, R1.1, R34.1, U14.6 (CG)
- net GEK100_KEY: now also U6.1 (KEY)
- net GEK100_RST: now also U6.3 (RST)
- net GND: now also C1.1, C10.1, C12.1, C15.1, C16.2, C2.1, C3.1, C30.1, C31.1, C43.2, C61.2, C62.1, C9.2, R1.2, R11.1, R12.1, R3.1, R5.1, R9.1, U14.5 (GND), U3.17 (PGND), U4.2 (GND), U5.2 (VSS), U6.2 (GND)
- net PWR_3V3_EN: now also R5.2, U4.1 (EN), U6.5 (OUTH)
- net STC3115_ALM: now also U14.1 (ALM)
- net VBAT: now also C10.2, C43.1, CN2.1, R2.2, U14.9 (VCC)
- net VCC: now also C1.2, C12.2, C15.2, C3.2, C30.2, C62.2, L2.2, U4.4 (VIN), U5.1 (VIN), U5.3 (CE), U6.6 (VDD)
- net VCC_1V8: now also C31.2, U5.5 (VOUT)
- net VCC_3V3: now also C2.2, L1.2, R4.2
- new net: R33.2, R34.2
- new net: C11.2, D2.2 (A), L2.1
- new net: R3.2, R4.1, U4.5 (FB)
- new net: C61.1, R2.1, U14.10 (VIN)
- new net: R33.1, U14.8 (BATD/CD)
- new net: R13.1, R15.1
- new net: R14.1, R16.1
- new net: L1.1, U4.3 (SW)
- new net STC3115_I2C_SCL: U14.3 (SCL)
- new net STC3115_I2C_SDA: U14.2 (SDA)
- new net VCC_PMID: C16.1, D2.1 (C)
Other:
- note removed: "GEK100 KEY has an internal 33k pull-up; RST has an internal 33k pull-down. KEY must connect to an external normally-open power button to GND. Select the GEK100 timing suffix explicitly before assembly (source note: GEK100-57)."
- company: ESP32-S31 MP3 -> (none)
- title: Charging and power rails -> (none)
