File: hardware-q2/3_DAC.kicad_sch (KiCad schematic)
At the start: 26 parts, among them CN1 PJ-342B-TX-SMT, U2 CS43131-CNZ, U7 PCA9306DQER, U8 SN74LV4T125RGYR, X1 26MHz

Commit message: feat: save finalized module mainboard and fabrication review
Parts:
- removed C17, C19, C20, C21, C22, C23, C24, C25: 2.2uF, MP3_Source:C0402_1, symbol MP3_Source:CL05A225MQ5NSNC
- removed C18, C8: 22uF, MP3_Source:C0603, symbol MP3_Source:CL10A226MQ8NRNC
- removed C26: 4.7uF, MP3_Source:C0402_1, symbol MP3_Source:CapAcitance_1
- removed C27, C28, C29: 100nF, MP3_Source:C0402_1, symbol MP3_Source:CapAcitance_1
- removed C32, C33: 10pF, MP3_Source:C0402_1, symbol MP3_Source:CC0402JRNPO9BN100
- removed C34: 100nF, MP3_Source:C0402_1, symbol MP3_Source:cl05b104ko5nnnc_2
- removed C35: 100nF, MP3_Source:C0402_1, symbol MP3_Source:cl05b104ko5nnnc_1
- removed CN1: PJ-342B-TX-SMT, MP3_Source:AUDIO-SMD_PJ-342B-TX-SMT, symbol MP3_Source:PJ-342B-TX-SMT
- removed R17: 200K, MP3_Source:R0402_2, symbol MP3_Source:0402WGF2003TCE
- removed R18, R19: 10K, MP3_Source:R0402_1, symbol MP3_Source:rc0402fr-071kl
- removed U2: CS43131-CNZ, MP3_Source:QFN-40_L5.0-W5.0-P0.40-TL-EP3.6_1, symbol MP3_Source:CS43131-CNZ_func
- removed U7: PCA9306DQER, MP3_Source:X2SON-8_L1.4-W1.0-P0.35-BL, symbol MP3_Source:PCA9306DQER
- removed U8: SN74LV4T125RGYR, MP3_Source:VQFN-14_L3.5-W3.5-P0.50-BL-EP, symbol MP3_Source:SN74LV4T125RGYR_self
- removed X1: 26MHz, MP3_Source:CRYSTAL-SMD_4P-L3.2-W2.5-BL_1, symbol MP3_Source:X322526MMB4SI
- added ?: (no value), ProPrj_esp-easyedapro:, symbol ProPrj_esp-easyedapro:Drawing-Symbol_A4
- added C17, C19, C20, C21, C22, C23, C24, C25: 2.2uF, ProPrj_esp-easyedapro:C0402_1, symbol ProPrj_esp-easyedapro:CL05A225MQ5NSNC
- added C18, C8: 22uF, ProPrj_esp-easyedapro:C0603, symbol ProPrj_esp-easyedapro:CL10A226MQ8NRNC
- added C26: 4.7uF, ProPrj_esp-easyedapro:C0603_1, symbol ProPrj_esp-easyedapro:CapAcitance_1
- added C27, C28, C29: 100nF, ProPrj_esp-easyedapro:C0603_1, symbol ProPrj_esp-easyedapro:CapAcitance_1
- added C32, C33: 10pF, ProPrj_esp-easyedapro:C0402_1, symbol ProPrj_esp-easyedapro:CC0402JRNPO9BN100
- added C34: 100nF, ProPrj_esp-easyedapro:, symbol ProPrj_esp-easyedapro:cl05b104ko5nnnc_2
- added C35: 100nF, ProPrj_esp-easyedapro:, symbol ProPrj_esp-easyedapro:cl05b104ko5nnnc_1
- added CN1: PJ-342B-TX-SMT, ProPrj_esp-easyedapro:AUDIO-SMD_PJ-342B-TX-SMT, symbol ProPrj_esp-easyedapro:PJ-342B-TX-SMT
- added R17: 200K, ProPrj_esp-easyedapro:R0402_2, symbol ProPrj_esp-easyedapro:0402WGF2003TCE
- added R18, R19: 10K, ProPrj_esp-easyedapro:, symbol ProPrj_esp-easyedapro:rc0402fr-071kl
- added U2: CS43131-CNZ, ProPrj_esp-easyedapro:QFN-40_L5.0-W5.0-P0.40-TL-EP3.6_1, symbol ProPrj_esp-easyedapro:CS43131-CNZ_func
- added U7: PCA9306DQER, ProPrj_esp-easyedapro:X2SON-8_L1.4-W1.0-P0.35-BL, symbol ProPrj_esp-easyedapro:PCA9306DQER
- added U8: SN74LV4T125RGYR, ProPrj_esp-easyedapro:VQFN-14_L3.5-W3.5-P0.50-BL-EP, symbol ProPrj_esp-easyedapro:SN74LV4T125RGYR_self
- added X1: 26MHz, ProPrj_esp-easyedapro:CRYSTAL-SMD_4P-L3.2-W2.5-BL_1, symbol ProPrj_esp-easyedapro:X322526MMB4SI
Connections:
- net CS43131_I2S_LRCK: now also U2.38 (LRCK1), U8.6 (2Y)
- net CS43131_I2S_SCLK: now also U2.34 (SCLK1), U8.8 (3Y)
- net CS43131_I2S_SDIN: now also U2.2 (SDIN1), U8.3 (1Y)
- net CS43131_RST#_1V8: now also U2.28 (RESET#), U8.11 (4Y)
- net CS43131_SCL_1V8: now also R18.1, U2.39 (SDA), U7.3 (SCL1)
- net CS43131_SDA_1V8: now also R19.1, U2.1 (SCL), U7.4 (SDA1)
- net DAC_I2C_SCL: now also U7.6 (SCL2)
- net DAC_I2C_SDA: now also U7.5 (SDA2)
- net DAC_I2S_LRCK: now also U8.5 (2A)
- net DAC_I2S_SCLK: now also U8.9 (3A)
- net DAC_I2S_SDIN: now also U8.2 (1A)
- net DAC_RST#: now also U8.12 (4A)
- net GND: now also C17.2, C19.2, C21.2, C22.2, C23.1, C26.2, C27.2, C28.2, C29.2, C34.2, C35.1, CN1.2, CN1.5, U2.13 (HPREFA), U2.17 (HPREFB), U2.19 (GNDCP), U2.30 (ADR), U2.35 (GNDD), U2.41 (EP), U2.8 (GNDA), U7.1 (GND), U8.1 (1OE#), U8.10 (3OE#), U8.13 (4OE#), U8.15 (GND), U8.4 (2OE#), U8.7 (GND), X1.2 (GND), X1.4 (GND)
- net VCC: now also C26.1, C29.1, U2.26 (VP)
- net VCC_1V8: now also C17.1, C23.2, C27.1, C28.1, C34.1, C35.2, C8.2, R18.2, R19.2, U2.25 (VCP), U2.31 (VL), U2.4 (VD), U2.7 (VA), U7.2 (VREF1), U8.14 (VCC)
- net VCC_3V3: now also R17.2
- new net: C20.1, U2.10 (FLYP_VA)
- new net: C20.2, U2.11 (FLYN_VA)
- new net: C21.1, U2.21 (VCP_FILT+)
- new net: C32.2, U2.36 (XTO), X1.1 (OSC1)
- new net: C33.1, U2.37 (XTI/MCLK), X1.3 (OSC2)
- new net: R17.1, U7.7 (VREF2), U7.8 (EN)
- new net: C32.1, C33.2
- new net: C18.2, C19.1, U2.9 (–VA)
- new net: C24.1, U2.24 (FLYP_VCP)
- new net: C24.2, C25.2, U2.23 (FLYC_VCP)
- new net: CN1.3, U2.14 (HPOUTA)
- new net: CN1.6, U2.16 (HPOUTB)
- new net: C22.1, U2.18 (VCP_FILT–)
- new net: C25.1, U2.20 (FLYN_VCP)
- new net: C8.1, U2.5 (FILT+)
- new net: C18.1, U2.6 (FILT-)
Other:
- company: ESP32-S31 MP3 -> (none)
- title: CS43131 audio DAC -> (none)
