File: hardware-q2/4_DISPLAY.kicad_sch (KiCad schematic)
At the start: 11 parts, among them U16 PAM2804AAB010

Commit message: feat: save finalized module mainboard and fabrication review
Parts:
- removed C42, C55, C56, C57: 10uF, MP3_Source:C0603_1, symbol MP3_Source:Capacitance
- removed C45, C46: 100nF, MP3_Source:C0402, symbol MP3_Source:Capacitance
- removed FPC2: 2.09寸320*375高清R角方屏QSPI, MP3_Source:CONN-TH-21P_AFE03-S21FMA-1H, symbol MP3_Source:AFE03-S21FMA-1H
- removed L4: 4.7uH, MP3_Source:IND-SMD_L2.0-W1.6, symbol MP3_Source:WPN201610M2R2MT
- removed R40: 1R5, MP3_Source:R1206, symbol MP3_Source:电阻
- removed R41: 100K, MP3_Source:R0402, symbol MP3_Source:电阻
- removed U16: PAM2804AAB010, MP3_Source:SOT-23-5_L3.0-W1.7-P0.95-LS2.8-BR, symbol MP3_Source:PAM2804AAB010
- added ?: (no value), ProPrj_esp-easyedapro:, symbol ProPrj_esp-easyedapro:Drawing-Symbol_A4
- added C42, C55, C56, C57: 10uF, ProPrj_esp-easyedapro:C0402, symbol ProPrj_esp-easyedapro:Capacitance
- added C45, C46: 100nF, ProPrj_esp-easyedapro:C0402, symbol ProPrj_esp-easyedapro:Capacitance
- added FPC2: 2.09寸320*375高清R角方屏QSPI, ProPrj_esp-easyedapro:CONN-TH-21P_AFE03-S21FMA-1H, symbol ProPrj_esp-easyedapro:AFE03-S21FMA-1H
- added L4: 4.7uH, ProPrj_esp-easyedapro:IND-SMD_L2.0-W1.6, symbol ProPrj_esp-easyedapro:WPN201610M2R2MT
- added R40: 1R5, ProPrj_esp-easyedapro:R1206, symbol ProPrj_esp-easyedapro:电阻
- added R41: 100K, ProPrj_esp-easyedapro:R1206, symbol ProPrj_esp-easyedapro:电阻
- added U16: PAM2804AAB010, ProPrj_esp-easyedapro:SOT-23-5_L3.0-W1.7-P0.95-LS2.8-BR, symbol ProPrj_esp-easyedapro:PAM2804AAB010
Connections:
- net GND: now also C42.1, C45.2, C46.2, C55.1, C56.1, C57.1, FPC2.12, FPC2.17, R40.1, R41.1, U16.2 (GND)
- net LCD_LEDA: now also C42.2, C55.2, FPC2.1, L4.2
- net LCD_LEDK: now also FPC2.2, R40.2, U16.5 (FB)
- net VCC_3V3: now also C45.1, C46.1, FPC2.13, FPC2.14
- net VCC_LCD_BG: now also C56.2, C57.2, U16.4 (VIN)
- new net: L4.1, U16.3 (SW)
- new net LCD_BG_PWM: R41.2, U16.1 (EN)
- new net LCD_CLK: FPC2.5
- new net LCD_CS: FPC2.7
- new net LCD_D0: FPC2.11
- new net LCD_D1: FPC2.10
- new net LCD_D2: FPC2.9
- new net LCD_D3: FPC2.8
- new net LCD_RST: FPC2.4
- new net LCD_TE: FPC2.3
- new net TP_INT: FPC2.21
- new net TP_RESET: FPC2.18
- new net TP_SCL: FPC2.19
- new net TP_SDA: FPC2.20
- no-connect marks 5 -> 3
Other:
- company: ESP32-S31 MP3 -> (none)
- title: QSPI display and backlight -> (none)
