File: hardware-q2/6_USB.kicad_sch (KiCad schematic)
At the start: 12 parts, among them U12 CH343P, U17 SGM7229YMS10G/TR

Commit message: feat: save finalized module mainboard and fabrication review
Parts:
- removed C36, C37, C38, C44: 100nF, MP3_Source:C0402, symbol MP3_Source:Capacitance
- removed D1: USBLC6-2SC6, MP3_Source:SOT-23-6_L2.9-W1.6-P0.95-LS2.8-BL, symbol MP3_Source:USBLC6-2SC6_C2687116
- removed R21, R22: 100K, MP3_Source:R0402, symbol MP3_Source:电阻
- removed R31, R32: 5K1, MP3_Source:R0402, symbol MP3_Source:电阻
- removed U12: CH343P, MP3_Source:TQFN-16_L3.0-W3.0-P0.50-BL-EP1.7, symbol MP3_Source:CH343P
- removed U17: SGM7229YMS10G/TR, MP3_Source:MSOP-10_L3.0-W3.0-P0.50-LS4.9-BL, symbol MP3_Source:SGM7229YMS10G/TR_C5153175
- removed USB1: TYPE-C 16PIN 2MD(073), MP3_Source:USB-C-SMD_TYPE-C-16PIN-2MD-073, symbol MP3_Source:TYPE-C 16PIN 2MD(073)
- added ?: (no value), ProPrj_esp-easyedapro:, symbol ProPrj_esp-easyedapro:Drawing-Symbol_A4
- added C36, C37, C38, C44, C51: 100nF, ProPrj_esp-easyedapro:C0402, symbol ProPrj_esp-easyedapro:Capacitance
- added D1: USBLC6-2SC6, ProPrj_esp-easyedapro:SOT-23-6_L2.9-W1.6-P0.95-LS2.8-BL, symbol ProPrj_esp-easyedapro:USBLC6-2SC6_C2687116
- added R21: 100K, ProPrj_esp-easyedapro:R1206, symbol ProPrj_esp-easyedapro:电阻
- added R31, R32: 5K1, ProPrj_esp-easyedapro:R1206, symbol ProPrj_esp-easyedapro:电阻
- added U12: CH343P, ProPrj_esp-easyedapro:TQFN-16_L3.0-W3.0-P0.50-BL-EP1.7, symbol ProPrj_esp-easyedapro:CH343P
- added U17: SGM7229YMS10G/TR, ProPrj_esp-easyedapro:MSOP-10_L3.0-W3.0-P0.50-LS4.9-BL, symbol ProPrj_esp-easyedapro:SGM7229YMS10G/TR_C5153175
- added USB1: TYPE-C 16PIN 2MD(073), ProPrj_esp-easyedapro:USB-C-SMD_TYPE-C-16PIN-2MD-073, symbol ProPrj_esp-easyedapro:TYPE-C 16PIN 2MD(073)
Connections:
- net CH343P_UART_DTR: now also U12.12 (DTRTNOW)
- net CH343P_UART_RTS: now also U12.13 (RTS)
- net CH343P_UART_RX: now also U12.5 (RXD)
- net CH343P_UART_TX: now also U12.4 (TXD)
- net CH343P_USB_DN: now also U12.8 (UD-), U17.8 (HSD2-)
- net CH343P_USB_DP: now also U12.7 (UD+), U17.9 (HSD2+)
- net GND: now also C36.2, C37.2, C38.2, C44.2, C51.2, D1.2 (GND), R21.1, R31.1, R32.1, U12.17 (EP), U12.2 (GND), U17.5 (GND), USB1.13 (EH), USB1.14 (EH), USB1.A1B12 (GND), USB1.B1A12 (GND)
- net TYPEC_USB_DN: now also D1.4 (I/O2), U17.4 (D-)
- net TYPEC_USB_DN_IN: now also D1.3 (I/O2), USB1.A7 (Dn1), USB1.B7 (Dn2)
- net TYPEC_USB_DP: now also D1.6 (I/O1), U17.3 (D+)
- net TYPEC_USB_DP_IN: now also D1.1 (I/O1), USB1.A6 (Dp1), USB1.B6 (Dp2)
- net VBUS_5V: now also C36.1, C44.1, C51.1, D1.5 (VBUS), U12.3 (VDD5), U12.9 (VBUS), U17.1 (VCC), USB1.A4B9 (VBUS), USB1.B4A9 (VBUS)
- net VCC_3V3: now also C37.1, U12.1 (VIO)
- new net: R31.2, USB1.A5 (CC1)
- new net: C38.1, U12.6 (V3)
- new net: R32.2, USB1.B5 (CC2)
- new net SGM7227_EN#: R21.2, U17.10 (OE#)
- new net SGM7227_SELECT: U17.2 (S)
- new net SGM7227_USB1_DN: U17.6 (HSD1-)
- new net SGM7227_USB1_DP: U17.7 (HSD1+)
Other:
- company: ESP32-S31 MP3 -> (none)
- title: USB-C and programming -> (none)
