File: hardware-q2/8_FLASH{slash}SDCARD.kicad_sch (KiCad schematic)
At the start: 9 parts, among them U1 RX8130CE:BB, U15 LSM6DS3TR-C

Commit message: feat: save finalized module mainboard and fabrication review
Parts:
- removed ?: (no value), ProPrj_esp-easyedapro:, symbol ProPrj_esp-easyedapro:Drawing-Symbol_A4
- removed C47, C48, C53, C6, C7: 100nF, ProPrj_esp-easyedapro:C0402, symbol ProPrj_esp-easyedapro:Capacitance
- removed C54: 1uF, ProPrj_esp-easyedapro:C0402, symbol ProPrj_esp-easyedapro:Capacitance
- removed U1: RX8130CE:BB, ProPrj_esp-easyedapro:RTC-SMD_L3.2-W2.5-P0.7-RX8130CE, symbol ProPrj_esp-easyedapro:RX8130CE{colon}BB
- removed U15: LSM6DS3TR-C, ProPrj_esp-easyedapro:LGA-14_L3.0-W2.5-P0.50-TL, symbol ProPrj_esp-easyedapro:LSM6DS3TR-C
- added ?: (no value), ProPrj_esp-easyedapro:, symbol ProPrj_esp-easyedapro:Drawing-Symbol_A4
- added C49: 10uF, ProPrj_esp-easyedapro:C0402, symbol ProPrj_esp-easyedapro:HGC0402R5106M100NTEJ
- added C50, C60: 100nF, ProPrj_esp-easyedapro:C0402, symbol ProPrj_esp-easyedapro:HGC0402R5106M100NTEJ
- added C52: 1uF, ProPrj_esp-easyedapro:C0402, symbol ProPrj_esp-easyedapro:HGC0402R5106M100NTEJ
- added CARD2: TF PUSH, ProPrj_esp-easyedapro:TF-SMD_TF-PUSH, symbol ProPrj_esp-easyedapro:TF PUSH
- added R47: 100K, ProPrj_esp-easyedapro:R1206, symbol ProPrj_esp-easyedapro:电阻
- added U13: W25Q128JVSIQ, ProPrj_esp-easyedapro:SOIC-8_L5.3-W5.3-P1.27-LS8.0-BL, symbol ProPrj_esp-easyedapro:W25Q128JVSIQTR
Connections:
- net GND: now also C49.1, C50.1, C52.1, C60.1, CARD2.10 (EP), CARD2.11 (EP), CARD2.12 (EP), CARD2.13 (EP), CARD2.6 (VSS), U13.4 (GND)
- net VCC_3V3: now also C49.2, C50.2, C52.2, CARD2.4 (VDD), U13.8 (VCC)
- new net: C60.2, R47.2
- new net FLASH_SPI_CLK: U13.6 (CLK)
- new net FLASH_SPI_CS: R47.1, U13.1 (CS#)
- new net FLASH_SPI_DI/IO1: U13.5 (DI)
- new net FLASH_SPI_DO/IO0: U13.2 (DO)
- new net FLASH_SPI_HOLD#/IO3: U13.7 (IO3)
- new net FLASH_SPI_WP#/IO2: U13.3 (IO2)
- new net SDCARD_CD_DET: CARD2.CD
- new net SDCARD_SDIO_CLK: CARD2.5 (CLX)
- new net SDCARD_SDIO_CMD: CARD2.3 (CMD)
- new net SDCARD_SDIO_DATA0: CARD2.7 (DAT0)
- new net SDCARD_SDIO_DATA1: CARD2.8 (DAT1)
- new net SDCARD_SDIO_DATA2: CARD2.1 (DAT2)
- new net SDCARD_SDIO_DATA3: CARD2.2 (CD/DAT3)
- no-connect marks 4 -> 0
Other:
- note added: "NC"
