File: hardware-q2/9_P1.kicad_sch (KiCad schematic)
At the start: 4 parts

Commit message: feat: save finalized module mainboard and fabrication review
Parts:
- removed SCREW1, SCREW2, SCREW4, SCREW5: M2 clearance 2.2mm, MP3_Source:MountingHole_2.2mm, symbol MP3_Source:螺丝孔
- added ? (x62): (no value), ProPrj_esp-easyedapro:, symbol ProPrj_esp-easyedapro:Short-Symbol-Auto
- added ?: (no value), ProPrj_esp-easyedapro:, symbol ProPrj_esp-easyedapro:Drawing-Symbol_A4
- added SCREW1, SCREW2, SCREW3, SCREW5: (no value), ProPrj_esp-easyedapro:M3螺丝, symbol ProPrj_esp-easyedapro:螺丝孔
Other:
- note added: "AUDIO DAC"
- note added: "ESP32S31"
- note added: "FLASH/SDCARD"
- note removed: "Board: 48.00 x 76.00 mm; corner radius 1.20 mm; six copper layers. Four M2 clearance holes, diameter 2.20 mm, NPTH. Original SCREW3 was outside the board edge and has been removed. Use the actual PCB hole coordinates for enclosure bosses; do not use source Gerber coordinates. Keep the ESP32 antenna area free of metal, battery foil and ground copper. The PCB size fits within a 50 x 80 mm envelope,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"
- note removed: "Mounting centers from PCB top-left (mm): SCREW1: X 3.0615 Y 69.9635 drill 2.20 NPTH SCREW2: X 11.5730 Y 34.3608 drill 2.20 NPTH SCREW4: X 45.8365 Y 34.7870 drill 2.20 NPTH SCREW5: X 10.8085 Y 3.7485 drill 2.20 NPTH USB-C footprint extends 1.22 mm beyond bottom edge. Headphone footprint extends 2.19 mm beyond bottom edge. Confirm connector STEP / datasheet dimensions before enclosure tooling."
- note removed: "PCB / enclosure interface"
- company: ESP32-S31 MP3 -> (none)
- title: Mechanical constraints -> (none)
