File: hardware-q2-v2/CORE_1.kicad_sch (KiCad schematic)
At the start: 21 parts, among them U10 W25Q128JVSIQ, Y101 40MHz 15pF 10ppm MDH 2.3.3.40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

Commit message: fix: standardize V2 0402 resistor and capacitor footprints
Parts:
- C101: footprint V2:FP_C101 -> V2:C_0402_1005Metric
- C102: footprint V2:FP_C102 -> V2:C_0402_1005Metric
- C105: footprint V2:FP_C105 -> V2:C_0402_1005Metric
- C106: footprint V2:FP_C106 -> V2:C_0402_1005Metric
- C110: footprint V2:FP_C110 -> V2:C_0402_1005Metric
- C113: footprint V2:FP_C113 -> V2:C_0402_1005Metric
- C114: footprint V2:FP_C114 -> V2:C_0402_1005Metric
- C115: footprint V2:FP_C115 -> V2:C_0402_1005Metric
- C116: footprint V2:FP_C116 -> V2:C_0402_1005Metric
- C117: footprint V2:FP_C117 -> V2:C_0402_1005Metric
- C118: footprint V2:FP_C118 -> V2:C_0402_1005Metric
- C119: footprint V2:FP_C119 -> V2:C_0402_1005Metric
- C120: footprint V2:FP_C120 -> V2:C_0402_1005Metric
- C121: footprint V2:FP_C121 -> V2:C_0402_1005Metric
- C122: footprint V2:FP_C122 -> V2:C_0402_1005Metric
- C123: footprint V2:FP_C123 -> V2:C_0402_1005Metric
- C124: footprint V2:FP_C124 -> V2:C_0402_1005Metric
- C125: footprint V2:FP_C125 -> V2:C_0402_1005Metric
