File: hardware-q2-v2/CORE_2.kicad_sch (KiCad schematic)
At the start: 19 parts

Commit message: fix: standardize V2 0402 resistor and capacitor footprints
Parts:
- R101: footprint V2:FP_R101 -> V2:R_0402_1005Metric
- R102: footprint V2:FP_R102 -> V2:R_0402_1005Metric
- R103: footprint V2:FP_R103 -> V2:R_0402_1005Metric
- R104: footprint V2:FP_R104 -> V2:R_0402_1005Metric
- R105: footprint V2:FP_R105 -> V2:R_0402_1005Metric
- R106: footprint V2:FP_R106 -> V2:R_0402_1005Metric
- R107: footprint V2:FP_R107 -> V2:R_0402_1005Metric
- R108: footprint V2:FP_R108 -> V2:R_0402_1005Metric
- R109: footprint V2:FP_R109 -> V2:R_0402_1005Metric
- R110: footprint V2:FP_R110 -> V2:R_0402_1005Metric
- R120: footprint V2:FP_R120 -> V2:R_0402_1005Metric
- R121: footprint V2:FP_R121 -> V2:R_0402_1005Metric
- R122: footprint V2:FP_R122 -> V2:R_0402_1005Metric
- R123: footprint V2:FP_R123 -> V2:R_0402_1005Metric
- R124: footprint V2:FP_R124 -> V2:R_0402_1005Metric
- R125: footprint V2:FP_R125 -> V2:R_0402_1005Metric
- R126: footprint V2:FP_R126 -> V2:R_0402_1005Metric
- R127: footprint V2:FP_R127 -> V2:R_0402_1005Metric
