File: hardware-q2-v2/CORE_RF_1.kicad_sch (KiCad schematic)
At the start: 9 parts

Commit message: fix: standardize V2 0402 resistor and capacitor footprints
Parts:
- C103: footprint V2:FP_C103 -> V2:C_0402_1005Metric
- C104: footprint V2:FP_C104 -> V2:C_0402_1005Metric
- C107: footprint V2:FP_C107 -> V2:C_0402_1005Metric
- C108: footprint V2:FP_C108 -> V2:C_0402_1005Metric
- C109: footprint V2:FP_C109 -> V2:C_0402_1005Metric
- L105: footprint V2:FP_L105 -> V2:R_0402_1005Metric
