File: hardware-q2-v2/DAC_1.kicad_sch (KiCad schematic)
At the start: 18 parts, among them CN1 PJ-342B-TX-SMT, U2 CS43131-CNZ, U7 PCA9306DQER, U8 SN74LV4T125RGYR, X1 26MHz

Commit message: fix: standardize V2 0402 resistor and capacitor footprints
Parts:
- C17: footprint V2:FP_C17 -> V2:C_0402_1005Metric
- C19: footprint V2:FP_C19 -> V2:C_0402_1005Metric
- C20: footprint V2:FP_C20 -> V2:C_0402_1005Metric
- C21: footprint V2:FP_C21 -> V2:C_0402_1005Metric
- C22: footprint V2:FP_C22 -> V2:C_0402_1005Metric
- C23: footprint V2:FP_C23 -> V2:C_0402_1005Metric
- C24: footprint V2:FP_C24 -> V2:C_0402_1005Metric
- C25: footprint V2:FP_C25 -> V2:C_0402_1005Metric
- C26: footprint V2:FP_C26 -> V2:C_0402_1005Metric
- C27: footprint V2:FP_C27 -> V2:C_0402_1005Metric
- C28: footprint V2:FP_C28 -> V2:C_0402_1005Metric
- C29: footprint V2:FP_C29 -> V2:C_0402_1005Metric
