File: hardware-q2-v2/DAC_2.kicad_sch (KiCad schematic)
At the start: 8 parts

Commit message: fix: standardize V2 0402 resistor and capacitor footprints
Parts:
- C32: footprint V2:FP_C32 -> V2:C_0402_1005Metric
- C33: footprint V2:FP_C33 -> V2:C_0402_1005Metric
- C34: footprint V2:FP_C34 -> V2:C_0402_1005Metric
- C35: footprint V2:FP_C35 -> V2:C_0402_1005Metric
- R17: footprint V2:FP_R17 -> V2:R_0402_1005Metric
- R18: footprint V2:FP_R18 -> V2:R_0402_1005Metric
- R19: footprint V2:FP_R19 -> V2:R_0402_1005Metric
