File: hardware-q2-v2/DISPLAY_1.kicad_sch (KiCad schematic)
At the start: 3 parts

Commit message: fix: standardize V2 0402 resistor and capacitor footprints
Parts:
- C136: footprint V2:FP_C136 -> V2:C_0402_1005Metric
- C137: footprint V2:FP_C137 -> V2:C_0402_1005Metric
