File: hardware-q2-v2/DOWNLOAD_1.kicad_sch (KiCad schematic)
At the start: 10 parts, among them Q106 MMBT3904, Q107 MMBT3904

Commit message: fix: standardize V2 0402 resistor and capacitor footprints
Parts:
- R132: footprint V2:FP_R132 -> V2:R_0402_1005Metric
- R133: footprint V2:FP_R133 -> V2:R_0402_1005Metric
