File: hardware-q2-v2/FLASH_SDCARD_1.kicad_sch (KiCad schematic)
At the start: 3 parts

Commit message: fix: standardize V2 0402 resistor and capacitor footprints
Parts:
- C49: footprint V2:FP_C49 -> V2:C_0402_1005Metric
- C50: footprint V2:FP_C50 -> V2:C_0402_1005Metric
