File: hardware-q2-v2/MCU_1.kicad_sch (KiCad schematic)
At the start: 21 parts

Commit message: fix: standardize V2 0402 resistor and capacitor footprints
Parts:
- C13: footprint V2:FP_C13 -> V2:C_0402_1005Metric
- C39: footprint V2:FP_C39 -> V2:C_0402_1005Metric
- R10: footprint V2:FP_R10 -> V2:R_0402_1005Metric
- R20: footprint V2:FP_R20 -> V2:R_0402_1005Metric
- R22: footprint V2:FP_R22 -> V2:R_0402_1005Metric
- R25: footprint V2:FP_R25 -> V2:R_0402_1005Metric
- R26: footprint V2:FP_R26 -> V2:R_0402_1005Metric
- R29: footprint V2:FP_R29 -> V2:R_0402_1005Metric
- R30: footprint V2:FP_R30 -> V2:R_0402_1005Metric
- R35: footprint V2:FP_R35 -> V2:R_0402_1005Metric
- R36: footprint V2:FP_R36 -> V2:R_0402_1005Metric
- R37: footprint V2:FP_R37 -> V2:R_0402_1005Metric
- R38: footprint V2:FP_R38 -> V2:R_0402_1005Metric
- R39: footprint V2:FP_R39 -> V2:R_0402_1005Metric
- R42: footprint V2:FP_R42 -> V2:R_0402_1005Metric
- R43: footprint V2:FP_R43 -> V2:R_0402_1005Metric
- R44: footprint V2:FP_R44 -> V2:R_0402_1005Metric
- R45: footprint V2:FP_R45 -> V2:R_0402_1005Metric
- R46: footprint V2:FP_R46 -> V2:R_0402_1005Metric
- R6: footprint V2:FP_R6 -> V2:R_0402_1005Metric
- R7: footprint V2:FP_R7 -> V2:R_0402_1005Metric
