File: hardware-q2-v2/MCU_2.kicad_sch (KiCad schematic)
At the start: 1 part

Commit message: fix: standardize V2 0402 resistor and capacitor footprints
Parts:
- R8: footprint V2:FP_R8 -> V2:R_0402_1005Metric
