File: hardware-q2-v2/MOTOR_1.kicad_sch (KiCad schematic)
At the start: 6 parts, among them CN3 Solder wire pads, U11 DRV2605LDGSR

Commit message: fix: standardize V2 0402 resistor and capacitor footprints
Parts:
- C4: footprint V2:FP_C4 -> V2:C_0402_1005Metric
- C5: footprint V2:FP_C5 -> V2:C_0402_1005Metric
- C58: footprint V2:FP_C58 -> V2:C_0402_1005Metric
