File: hardware-q2-v2/POWER_1.kicad_sch (KiCad schematic)
At the start: 18 parts, among them CN2 Solder wire pads, U14 STC3115AIQT, U3 DSCB_BQ25895RTW, U4 TLV62568DBVR, U5 ME6211C18M5G-N, U6 GEK100

Commit message: fix: standardize V2 0402 resistor and capacitor footprints
Parts:
- C11: footprint V2:FP_C11 -> V2:C_0402_1005Metric
- C3: footprint V2:FP_C3 -> V2:C_0402_1005Metric
- C30: footprint V2:FP_C30 -> V2:C_0402_1005Metric
- C31: footprint V2:FP_C31 -> V2:C_0402_1005Metric
- C43: footprint V2:FP_C43 -> V2:C_0402_1005Metric
