File: hardware-q2-v2/POWER_2.kicad_sch (KiCad schematic)
At the start: 17 parts

Commit message: fix: standardize V2 0402 resistor and capacitor footprints
Parts:
- C61: footprint V2:FP_C61 -> V2:C_0402_1005Metric
- R11: footprint V2:FP_R11 -> V2:R_0402_1005Metric
- R12: footprint V2:FP_R12 -> V2:R_0402_1005Metric
- R13: footprint V2:FP_R13 -> V2:R_0402_1005Metric
- R14: footprint V2:FP_R14 -> V2:R_0402_1005Metric
- R2: footprint V2:FP_R2 -> V2:R_0402_1005Metric
- R3: footprint V2:FP_R3 -> V2:R_0402_1005Metric
- R33: footprint V2:FP_R33 -> V2:R_0402_1005Metric
- R34: footprint V2:FP_R34 -> V2:R_0402_1005Metric
- R4: footprint V2:FP_R4 -> V2:R_0402_1005Metric
- R5: footprint V2:FP_R5 -> V2:R_0402_1005Metric
- R9: footprint V2:FP_R9 -> V2:R_0402_1005Metric
