File: hardware-q2-v2/POWER_AON_1.kicad_sch (KiCad schematic)
At the start: 17 parts, among them Q101 BSS138, Q102 BSS138, Q103 BSS138, Q104 BSS138, Q105 BSS138, U20 TLV75533PDBVR, U21 SN74LVC1G123DCUR

Commit message: fix: standardize V2 0402 resistor and capacitor footprints
Parts:
- C130: footprint V2:FP_C130 -> V2:C_0402_1005Metric
- C131: footprint V2:FP_C131 -> V2:C_0402_1005Metric
- C132: footprint V2:FP_C132 -> V2:C_0402_1005Metric
- C133: footprint V2:FP_C133 -> V2:C_0402_1005Metric
- C134: footprint V2:FP_C134 -> V2:C_0402_1005Metric
- C135: footprint V2:FP_C135 -> V2:C_0402_1005Metric
- R128: footprint V2:FP_R128 -> V2:R_0402_1005Metric
- R129: footprint V2:FP_R129 -> V2:R_0402_1005Metric
- R130: footprint V2:FP_R130 -> V2:R_0402_1005Metric
- R131: footprint V2:FP_R131 -> V2:R_0402_1005Metric
