File: hardware-q2-v2/SENSOR_1.kicad_sch (KiCad schematic)
At the start: 8 parts, among them U1 RX8130CE:BB, U15 LSM6DS3TR-C

Commit message: fix: standardize V2 0402 resistor and capacitor footprints
Parts:
- C47: footprint V2:FP_C47 -> V2:C_0402_1005Metric
- C48: footprint V2:FP_C48 -> V2:C_0402_1005Metric
- C53: footprint V2:FP_C53 -> V2:C_0402_1005Metric
- C54: footprint V2:FP_C54 -> V2:C_0402_1005Metric
- C6: footprint V2:FP_C6 -> V2:C_0402_1005Metric
- C7: footprint V2:FP_C7 -> V2:C_0402_1005Metric
