File: hardware-q2-v2/TOUCH_WHEEL_1.kicad_sch (KiCad schematic)
At the start: 2 parts

Commit message: fix: standardize V2 0402 resistor and capacitor footprints
Parts:
- C59: footprint V2:FP_C59 -> V2:C_0402_1005Metric
