File: hardware-q2-v2/USB_1.kicad_sch (KiCad schematic)
At the start: 12 parts, among them U12 CH343P, U17 SGM7229YMS10G/TR

Commit message: fix: standardize V2 0402 resistor and capacitor footprints
Parts:
- C36: footprint V2:FP_C36 -> V2:C_0402_1005Metric
- C37: footprint V2:FP_C37 -> V2:C_0402_1005Metric
- C38: footprint V2:FP_C38 -> V2:C_0402_1005Metric
- C44: footprint V2:FP_C44 -> V2:C_0402_1005Metric
- C51: footprint V2:FP_C51 -> V2:C_0402_1005Metric
- R21: footprint V2:FP_R21 -> V2:R_0402_1005Metric
- R31: footprint V2:FP_R31 -> V2:R_0402_1005Metric
- R32: footprint V2:FP_R32 -> V2:R_0402_1005Metric
